Commit message: codigo ICP ainda em debug

File: SC-LIO-SAM/SC-LIO-SAM/launch/include/config/GEORGIA_TECH.urdf (robot description, URDF)
Before this commit: robot GEORGIA_TECH_ROBOT, 3 links, 2 joints
Joints:
- joint imu_link_joint: origin xyz=0 0 0 rpy=0 0 0 -> xyz=0 0 0 rpy=-3.137 0 0

Commit message: GEORGIA TECH UPDATES

File: SC-LIO-SAM/SC-LIO-SAM/launch/include/config/GEORGIA_TECH.urdf (robot description, URDF)
Before this commit: robot GEORGIA_TECH_ROBOT, 3 links, 2 joints
Links:
- removed link sbg
Joints:
- removed joint imu_link_joint
- joint velo_base_link_joint: origin xyz=0 0 0 rpy=0 0 0 -> xyz=0.25 0 0.27 rpy=0 0 0
